File: ConFLiCTuino.sch (EAGLE design)
At the start: 73 parts, among them IC4 LM358D, J1 Power, Q1 IRLR024N, Q2 BC847B, Q3 BC847B, Q5 IRLR024N, Q6 IRLR024N, Q7 IRF9Z34NS, Q8 IRF9Z34NS

Commit message: init V0.3
Parts:
- D1, D3: value 1N400X -> S1D; device diode:DIODE-MELF-MLL41 -> diode:DIODE-DO214AC
Changed lines of the file:
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@@
 <grid distance="0.1" unitdist="inch" unit="inch" style="lines" multiple="1" display="no" altdistance="0.01" altunitdist="inch" altunit="inch"/>
 <layers>
-<layer number="1" name="Top" color="4" fill="1" visible="no" active="no"/>
-<layer number="2" name="Route2" color="1" fill="3" visible="no" active="no"/>
-<layer number="3" name="Route3" color="4" fill="3" visible="no" active="no"/>
-<layer number="4" name="Route4" color="1" fill="4" visible="no" active="no"/>
-<layer number="5" name="Route5" color="4" fill="4" visible="no" active="no"/>
-<layer number="6" name="Route6" color="1" fill="8" visible="no" active="no"/>
-<layer number="7" name="Route7" color="4" fill="8" visible="no" active="no"/>
-<layer number="8" name="Route8" color="1" fill="2" visible="no" active="no"/>
-<layer number="9" name="Route9" color="4" fill="2" visible="no" active="no"/>
-<layer number="10" name="Route10" color="1" fill="7" visible="no" active="no"/>
-<layer number="11" name="Route11" color="4" fill="7" visible="no" active="no"/>
-<layer number="12" name="Route12" color="1" fill="5" visible="no" active="no"/>
-<layer number="13" name="Route13" color="4" fill="5" visible="no" active="no"/>
-<layer number="14" name="Route14" color="1" fill="6" visible="no" active="no"/>
-<layer number="15" name="Route15" color="4" fill="6" visible="no" active="no"/>
-<layer number="16" name="Bottom" color="1" fill="1" visible="no" active="no"/>
-<layer number="17" name="Pads" color="2" fill="1" visible="no" active="no"/>
-<layer number="18" name="Vias" color="2" fill="1" visible="no" active="no"/>
-<layer number="19" name="Unrouted" color="6" fill="1" visible="no" active="no"/>
-<layer number="20" name="Dimension" color="15" fill="1" visible="no" active="no"/>
-<layer number="21" name="tPlace" color="7" fill="1" visible="no" active="no"/>
-<layer number="22" name="bPlace" color="7" fill="1" visible="no" active="no"/>
-<layer number="23" name="tOrigins" color="15" fill="1" visible="no" active="no"/>
-<layer number="24" name="bOrigins" color="15" fill="1" visible="no" active="no"/>
-<layer number="25" name="tNames" color="7" fill="1" visible="no" active="no"/>
-<layer number="26" name="bNames" color="7" fill="1" visible="no" active="no"/>
-<layer number="27" name="tValues" color="7" fill="1" visible="no" active="no"/>
-<layer number="28" name="bValues" color="7" fill="1" visible="no" active="no"/>
+<layer number="1" name="Top" color="4" fill="1" visible="yes" active="no"/>
+<layer number="2" name="Route2" color="1" fill="3" visible="yes" active="no"/>
+<layer number="3" name="Route3" color="4" fill="3" visible="yes" active="no"/>
+<layer number="4" name="Route4" color="1" fill="4" visible="yes" active="no"/>
+<layer number="5" name="Route5" color="4" fill="4" visible="yes" active="no"/>
+<layer number="6" name="Route6" color="1" fill="8" visible="yes" active="no"/>
+<layer number="7" name="Route7" color="4" fill="8" visible="yes" active="no"/>
+<layer number="8" name="Route8" color="1" fill="2" visible="yes" active="no"/>
+<layer number="9" name="Route9" color="4" fill="2" visible="yes" active="no"/>
+<layer number="10" name="Route10" color="1" fill="7" visible="yes" active="no"/>
+<layer number="11" name="Route11" color="4" fill="7" visible="yes" active="no"/>
+<layer number="12" name="Route12" color="1" fill="5" visible="yes" active="no"/>
+<layer number="13" name="Route13" color="4" fill="5" visible="yes" active="no"/>
+<layer number="14" name="Route14" color="1" fill="6" visible="yes" active="no"/>
+<layer number="15" name="Route15" color="4" fill="6" visible="yes" active="no"/>
+<layer number="16" name="Bottom" color="1" fill="1" visible="yes" active="no"/>
+<layer number="17" name="Pads" color="2" fill="1" visible="yes" active="no"/>
+<layer number="18" name="Vias" color="2" fill="1" visible="yes" active="no"/>
+<layer number="19" name="Unrouted" color="6" fill="1" visible="yes" active="no"/>
+<layer number="20" name="Dimension" color="15" fill="1" visible="yes" active="no"/>
+<layer number="21" name="tPlace" color="7" fill="1" visible="yes" active="no"/>
+<layer number="22" name="bPlace" color="7" fill="1" visible="yes" active="no"/>
+<layer number="23" name="tOrigins" color="15" fill="1" visible="yes" active="no"/>
+<layer number="24" name="bOrigins" color="15" fill="1" visible="yes" active="no"/>
+<layer number="25" name="tNames" color="7" fill="1" visible="yes" active="no"/>
+<layer number="26" name="bNames" color="7" fill="1" visible="yes" active="no"/>
+<layer number="27" name="tValues" color="7" fill="1" visible="yes" active="no"/>
+<layer number="28" name="bValues" color="7" fill="1" visible="yes" active="no"/>
 <layer number="29" name="tStop" color="7" fill="3" visible="no" active="no"/>
 <layer number="30" name="bStop" color="7" fill="6" visible="no" active="no"/>
@@
 <layer number="35" name="tGlue" color="7" fill="4" visible="no" active="no"/>
 <layer number="36" name="bGlue" color="7" fill="5" visible="no" active="no"/>
-<layer number="37" name="tTest" color="7" fill="1" visible="no" active="no"/>
-<layer number="38" name="bTest" color="7" fill="1" visible="no" active="no"/>
+<layer number="37" name="tTest" color="7" fill="1" visible="yes" active="no"/>
+<layer number="38" name="bTest" color="7" fill="1" visible="yes" active="no"/>
 <layer number="39" name="tKeepout" color="4" fill="11" visible="no" active="no"/>
 <layer number="40" name="bKeepout" color="1" fill="11" visible="no" active="no"/>
@@
 <layer number="44" name="Drills" color="7" fill="1" visible="no" active="no"/>
 <layer number="45" name="Holes" color="7" fill="1" visible="no" active="no"/>
-<layer number="46" name="Milling" color="3" fill="1" visible="no" active="no"/>
-<layer number="47" name="Measures" color="7" fill="1" visible="no" active="no"/>
-<layer number="48" name="Document" color="7" fill="1" visible="no" active="no"/>
-<layer number="49" name="Reference" color="7" fill="1" visible="no" active="no"/>
-<layer number="50" name="dxf" color="7" fill="1" visible="no" active="no"/>
-<layer number="51" name="tDocu" color="7" fill="1" visible="no" active="no"/>
-<layer number="52" name="bDocu" color="7" fill="1" visible="no" active="no"/>
+<layer number="46" name="Milling" color="3" fill="1" visible="yes" active="no"/>
+<layer number="47" name="Measures" color="7" fill="1" visible="yes" active="no"/>
+<layer number="48" name="Document" color="7" fill="1" visible="yes" active="no"/>
+<layer number="49" name="Reference" color="7" fill="1" visible="yes" active="no"/>
+<layer number="50" name="dxf" color="7" fill="1" visible="yes" active="no"/>
+<layer number="51" name="tDocu" color="7" fill="1" visible="yes" active="no"/>
+<layer number="52" name="bDocu" color="7" fill="1" visible="yes" active="no"/>
 <layer number="91" name="Nets" color="2" fill="1" visible="yes" active="yes"/>
 <layer number="92" name="Busses" color="1" fill="1" visible="yes" active="yes"/>
@@
 <part name="TEMP" library="pinhead" deviceset="PINHD-2X7" device=""/>
 <part name="R9" library="rcl" deviceset="R-EU_" device="M0805" value="10k NTC 3730K"/>
-<part name="D1" library="diode" deviceset="DIODE-" device="MELF-MLL41" value="1N400X"/>
-<part name="D3" library="diode" deviceset="DIODE-" device="MELF-MLL41" value="1N400X"/>
+<part name="D1" library="diode" deviceset="DIODE-" device="DO214AC" value="S1D"/>
+<part name="D3" library="diode" deviceset="DIODE-" device="DO214AC" value="S1D"/>
 <part name="LED" library="pinhead" deviceset="PINHD-2X4" device=""/>
 <part name="P+18" library="supply1" deviceset="+5V" device=""/>

Commit message: Init V0.4
Changed whole layout. More resistor nets and smaller board.
Parts:
- removed J1: Power, con-amp:FLOP-4W827001
- removed JP1: (no value), pinhead:PINHD-1X1
- removed R1, R3, R5, R7: 10k, rcl:R-EU_M0805
- removed R2, R4, R6, R8: 4k7, rcl:R-EU_M0805
- removed R20, R21, R22: 180, rcl:R-EU_M0805
- added PWR: (no value), con-amp:FLOPPY-4350211
- added RN2: 10K, resistor-dil:4R-NCAT16
- added RN3: 4k7, resistor-dil:4R-NCAT16
- added RN5: 220, resistor-dil:4R-NCAT16
- C49, C53: value 10p -> 22p
- IC1: value (none) -> MEGAARDUINO_CUSTOM; device arduino:MEGAARDUINO_13 -> arduino:MEGAARDUINO_CUSTOM
Connections:
- new net N$44: C6.2, IC1G$5.GND
- net +12V: now also IC1G$3.+VIN, PWR.1; no longer IC1.+VIN, J1.1
- net +3V3: now also IC1G$4.+3V3; no longer IC1.+3V3
- net +5V: now also IC1G$6.+5V, IC1G$7.+5V; no longer IC1.+5V@2, IC1.+5V@3
- net A_1: now also IC1G$1.(OC0A/OC1C/PCINT7)PB7; no longer IC1.(OC0A/OC1C/PCINT7)PB7
- net A_2: now also IC1G$1.(OC1B/PCINT6)PB6; no longer IC1.(OC1B/PCINT6)PB6
- net DFM: now also IC1G$1.PL1(ICP5); no longer IC1.PL1(ICP5)
- net GND: now also C54.1, IC1G$3.GND, IC1G$4.GND, IC1G$6.GND, IC1G$7.GND, PWR.2, PWR.3; no longer C54.2, C6.2, IC1.GND@1, IC1.GND@2, IC1.GND@3, IC1.GND@4, IC1.GND@5, J1.2, J1.3
- net LED_1: now also IC1G$1.PH6(OC2B), RN5D.2; no longer IC1.PH6(OC2B), R22.2
- net LED_2: now also IC1G$1.(OC2A/PCINT4)PB4, RN5C.2; no longer IC1.(OC2A/PCINT4)PB4, R21.2
- net LED_3: now also IC1G$1.(OC1A/PCINT5)PB5, RN5B.2; no longer IC1.(OC1A/PCINT5)PB5, R20.2
- net N$1: now also IC1G$1.(SDA/INT1)PD1; no longer IC1.(SDA/INT1)PD1
- net N$10: now also IC1G$1.(A15)PC7; no longer IC1.(A15)PC7
- net N$12: now also RN2B.2, RN3C.2; no longer R5.1, R6.1
- net N$13: now also IC1G$1.(A14)PC6; no longer IC1.(A14)PC6
- net N$14: now also RN2A.2, RN3D.2; no longer R7.1, R8.1
- net N$15: now also IC1G$1.(A13)PC5; no longer IC1.(A13)PC5
- net N$17: now also IC1G$1.(A12)PC4; no longer IC1.(A12)PC4
- net N$2: now also RN2D.2, RN3A.2; no longer R1.1, R2.1
- net N$23: now also IC1G$1.(A11)PC3; no longer IC1.(A11)PC3
- net N$26: now also IC1G$1.(A10)PC2; no longer IC1.(A10)PC2
- net N$27: now also IC1G$1.(A9)PC1; no longer IC1.(A9)PC1
- net N$28: now also IC1G$1.(A8)PC0; no longer IC1.(A8)PC0
- net N$29: now also IC1G$1.(SCK/PCINT1)PB1; no longer IC1.(SCK/PCINT1)PB1
- net N$30: now also IC1G$1.(SS/PCINT0)PB0; no longer IC1.(SS/PCINT0)PB0
- net N$31: now also IC1G$1.(MISO/PCINT3)PB3; no longer IC1.(MISO/PCINT3)PB3
- net N$32: now also IC1G$1.(MOSI/PCINT2)PB2; no longer IC1.(MOSI/PCINT2)PB2
- net N$33: now also IC1G$1.PF0(ADC0); no longer IC1.PF0(ADC0)
- net N$34: now also IC1G$1.PF1(ADC1); no longer IC1.PF1(ADC1)
- net N$35: now also IC1G$1.PF2(ADC2); no longer IC1.PF2(ADC2)
- net N$36: now also IC1G$1.PF3(ADC3); no longer IC1.PF3(ADC3)
- net N$37: now also IC1G$1.PF4(ADC4/TCK); no longer IC1.PF4(ADC4/TCK)
- net N$38: now also IC1G$1.PF5(ADC5/TMS); no longer IC1.PF5(ADC5/TMS)
- net N$39: now also IC1G$1.PF6(ADC6/TDO); no longer IC1.PF6(ADC6/TDO)
- net N$4: now also IC1G$1.PH1(TXD2); no longer IC1.PH1(TXD2)
- net N$40: now also IC1G$1.PF7(ADC7/TDI); no longer IC1.PF7(ADC7/TDI)
- net N$41: now also IC1G$1.PH3(OC4A); no longer IC1.PH3(OC4A)
- net N$43: now also IC1G$1.AREF; no longer IC1.AREF
- net N$5: now also RN2C.2, RN3B.2; no longer R3.1, R4.1
- net N$53: now also R26.1; no longer R26.2
- net N$54: now also C54.2, R26.2; no longer C54.1, R26.1
- net N$7: now also IC1G$1.(SCL/INT0)PD0; no longer IC1.(SCL/INT0)PD0
- net N$82: now also RN5B.1; no longer R20.1
- net N$83: now also RN5C.1; no longer R21.1
- net N$84: now also RN5D.1; no longer R22.1
- net N$9: now also IC1G$1.PH0(RXD2); no longer IC1.PH0(RXD2)
- net PWM_1: now also IC1G$1.PH5(OC4C); no longer IC1.PH5(OC4C)
- net PWM_2: now also IC1G$1.PH4(OC4B); no longer IC1.PH4(OC4B)
- net S$2: now also IC1G$5.+5V; no longer IC1.+5V@1
- net T_A_1: now also IC1G$1.(RXD1/INT2)PD2, RN2D.1; no longer IC1.(RXD1/INT2)PD2, R1.2
- net T_A_2: now also IC1G$1.(TXD1/INT3)PD3, RN2C.1; no longer IC1.(TXD1/INT3)PD3, R3.2
- net T_PWM_1: now also IC1G$1.(OC3C/INT5)PE5, RN2B.1; no longer IC1.(OC3C/INT5)PE5, R5.2
- net T_PWM_2: now also IC1G$1.(OC3B/INT4)PE4, RN2A.1; no longer IC1.(OC3B/INT4)PE4, R7.2
- net V+: now also IC1G$2.IOREF, RN3A.1, RN3B.1, RN3C.1, RN3D.1; no longer JP1.1, R2.2, R4.2, R6.2, R8.2
Other:
- note added: "This shield is for an Arduino Mega 2560."
- note removed: "IOREF"
- note removed: "This shield can be used with an Arduino Mega 2560 without modifications."
- moved on the sheet: C14, C15, C16, C17, C18, C19, C20, C21, C28, C6, EXT-1, EXT-10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
