File: ConFLiCTuino.sch (EAGLE design)
At the start: 67 parts, among them IC1 MEGAARDUINO_CUSTOM, IC4 LM358D, Q1 IRLR024N, Q2 BC847B, Q3 BC847B, Q5 IRLR024N, Q6 IRLR024N, Q7 IRF9Z34NS, Q8 IRF9Z34NS

Commit message: Changed some packages
Parts:
- R1, R12, R13, R16, R23, R24, R25, R26, R27: device rcl:R-EU_M0805 -> rcl:R-EU_0207/10
Other:
- moved on the sheet: RN5D
