File: ConFLiCTuino.brd (EAGLE design)
At the start: 86.4 x 53.3 mm, 67 parts, among them IC1 MEGAARDUINO_CUSTOM, IC4 LM358D, Q1 IRLR024N, Q2 BC847B, Q3 BC847B, Q5 IRLR024N, Q6 IRLR024N, Q7 IRF9Z34NS, Q8 IRF9Z34NS

Commit message: init V0.6
Changed 4-Pol PWM connectors to Molex-Footprint with hole for the kex
pin.
Parts:
- PWM1, PWM2: value 22-27-2041-04 -> 47053-1000; device con-molex:6410-04 -> con-molex:47053-1000
- moved Q2 2.06 mm to (60.0, 35.1)
- moved Q3 2.06 mm to (66.7, 35.1)
- moved R14 1.72 mm to (60.0, 38.9), turned to 180 degrees
- moved R15 1.72 mm to (66.7, 38.9), turned to 180 degrees
- moved PWM1 1.00 mm to (59.7, 24.1)
- moved PWM2 1.00 mm to (66.4, 24.1)
Routing:
- net N$22: track 3.03 -> 6.18 mm
- net N$25: track 3.03 -> 6.18 mm
- net PWM_2: track 43.2 -> 40.8 mm
- net PWM_1: track 38.2 -> 35.8 mm
- net N$12: track 45.3 -> 46.6 mm
- net N$14: track 39.9 -> 41.2 mm
- net +12V: track 121.5 -> 120.7 mm
Other:
- board text added: "0.6"
- board text removed: "0.5"
